File: _autosave-CAN to WIFI.kicad_pcb (KiCad board)
At the start: 2 copper layers, 48.2 x 54 mm, 68 parts, among them J1 C-OBD-II-16M, J2 USB_C_Receptacle_USB2.0_16P, J3 Conn_01x03_Pin, Q1 SS8050, Q2 SS8050, SW1 SW_Push, SW2 SW_Push, SW3 SW_Push, U1 MP2338GTL-P, U2 ESP32-WROOM-32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

Commit message: Update KiCad project files
Routing:
- net GND: track 0.00 -> 127.9 mm
- net V_BATT: track 0.00 -> 23.8 mm
- net Net-(Q1-E): track 0.00 -> 22.1 mm
- net Net-(J1-Pad5): track 0.00 -> 21.0 mm
- net Net-(U1-SW): track 0.00 -> 20.8 mm
- net Net-(J2-GND-PadA1): track 0.00 -> 18.6 mm
- net EN: track 0.00 -> 18.6 mm
- net Net-(C10-Pad1): track 0.00 -> 18.1 mm
- net Net-(Q2-E): track 0.00 -> 16.7 mm
- net Net-(U2-IO35): track 0.00 -> 16.6 mm
- net +5V: track 0.00 -> 12.6 mm
- net Net-(C13-Pad2): track 0.00 -> 11.6 mm
- net CAN_3V3: track 0.00 -> 10.8 mm
- net ESP_3V3: track 0.00 -> 10.3 mm
- net /MCU/WIFI/LED: track 0.00 -> 10.2 mm
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
Commit message: Update KiCad project files
Routing:
- net CAN_RX: track 0.00 -> 19.0 mm
- net CAN_TX: track 0.00 -> 9.79 mm
- net /MCU/COMM/LED: track 4.96 -> 0.00 mm
Changed lines of the file:
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@@
-	)
-	(segment
-		(start 132.301 80.301)
-		(end 132.301 78.126)
-		(width 0.2)
-		(layer "F.Cu")
-		(net 57)
-	)
-	(segment
-		(start 133.5 81.5)
-		(end 132.301 80.301)
-		(width 0.2)
-		(layer "F.Cu")
-		(net 57)
-	)
-	(segment
-		(start 132.2 78.025)
-		(end 131.25 78.025)
-		(width 0.2)
-		(layer "F.Cu")
-		(net 57)
-	)
-	(segment
-		(start 132.301 78.126)
-		(end 132.2 78.025)
-		(width 0.2)
-		(layer "F.Cu")
-		(net 57)
 	)
 	(segment
@@
 	)
 	(segment
+		(start 141.026 88.988064)
+		(end 140.014064 90)
+		(width 0.2)
+		(layer "F.Cu")
+		(net 84)
+	)
+	(segment
+		(start 140.014064 90)
+		(end 138.677 90)
+		(width 0.2)
+		(layer "F.Cu")
+		(net 84)
+	)
+	(segment
+		(start 141.026 84.406)
+		(end 141.026 88.988064)
+		(width 0.2)
+		(layer "F.Cu")
+		(net 84)
+	)
+	(segment
+		(start 138.677 90)
+		(end 131.782 83.105)
+		(width 0.2)
+		(layer "F.Cu")
+		(net 84)
+	)
+	(segment
+		(start 140.025 83.405)
+		(end 141.026 84.406)
+		(width 0.2)
+		(layer "F.Cu")
+		(net 84)
+	)
+	(segment
+		(start 131.782 83.105)
+		(end 131.25 83.105)
+		(width 0.2)
+		(layer "F.Cu")
+		(net 84)
+	)
+	(segment
+		(start 139.594 80.026)
+		(end 132.931 80.026)
+		(width 0.2)
+		(layer "F.Cu")
+		(net 88)
+	)
+	(segment
+		(start 140.025 79.595)
+		(end 139.594 80.026)
+		(width 0.2)
+		(layer "F.Cu")
+		(net 88)
+	)
+	(segment
+		(start 132.931 80.026)
+		(end 132.2 79.295)
+		(width 0.2)
+		(layer "F.Cu")
+		(net 88)
+	)
+	(segment
+		(start 132.2 79.295)
+		(end 131.25 79.295)
+		(width 0.2)
+		(layer "F.Cu")
+		(net 88)
+	)
+	(segment
+		(start 130.718 79.295)
+		(end 131.25 79.295)
+		(width 0.2)
+		(layer "F.Cu")
+		(net 88)
+	)
+	(segment
